File: LM317_3S_LithiumCharger_2018_05_13.brd (EAGLE design)
At the start: 58.3 x 35.2 mm, 27 parts, among them Q2 MOSFET-NCHANNELBSS123LT1G, Q3 MOSFET-PCHANNEL, U1 LD1086BV

Commit message: Add files via upload
Parts:
- moved C2 1.52 mm to (46.0, 20.3)
- moved U1 1.27 mm to (54.9, 38.1)
- moved Q1 1.27 mm to (71.4, 38.1)
Routing:
- net VREG: track 30.0 -> 33.6 mm
- net VBATT: track 31.1 -> 29.7 mm
- net ENABLE: track 57.0 -> 55.7 mm
- net VIN: track 75.9 -> 75.0 mm
- net N$2: track 14.1 -> 14.7 mm
Other:
- board size 58.3 x 35.2 mm -> 58.1 x 34.9 mm
- board text added: "12.6V Lithium Charger With Autoshut off 5/13/2018 Chris S"
- board text removed: "12.6V Lithium Charger With Charging, Done and Autoshut off 5/13/2018 Chris S"
Changed lines of the file:
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@@
 <plain>
 <wire x1="35.56" y1="4.445" x2="93.65" y2="4.445" width="0" layer="20"/>
-<wire x1="93.65" y1="4.445" x2="93.904" y2="39.614" width="0" layer="20"/>
-<wire x1="93.904" y1="39.614" x2="35.814" y2="39.614" width="0" layer="20"/>
-<wire x1="35.814" y1="39.614" x2="35.56" y2="4.445" width="0" layer="20"/>
+<wire x1="93.65" y1="4.445" x2="93.65" y2="39.36" width="0" layer="20"/>
+<wire x1="93.65" y1="39.36" x2="35.56" y2="39.36" width="0" layer="20"/>
+<wire x1="35.56" y1="39.36" x2="35.56" y2="4.445" width="0" layer="20"/>
 <text x="69.85" y="6.35" size="0.8128" layer="25" ratio="1">DONE</text>
 <text x="55.245" y="6.35" size="0.8128" layer="25" ratio="1">CHARGING</text>
@@
 <hole x="37.465" y="6.35" drill="3.2"/>
 <hole x="91.44" y="6.35" drill="3.2"/>
-<text x="37.846" y="11.049" size="1.016" layer="25" ratio="1">12.6V Lithium Charger
-With Charging, Done and Autoshut off
+<text x="36.322" y="25.019" size="1.016" layer="25" ratio="1">12.6V Lithium Charger
+With Autoshut off
 5/13/2018
 Chris S</text>
-<text x="42.545" y="20.955" size="1.016" layer="25" ratio="1">-</text>
+<text x="42.545" y="21.209" size="1.016" layer="25" ratio="1">-</text>
 <text x="38.1" y="23.495" size="1.016" layer="25" ratio="1">VIN</text>
 <text x="88.265" y="23.495" size="1.016" layer="25" ratio="1">VBATT</text>
 <text x="86.36" y="18.415" size="1.016" layer="25" ratio="1">-</text>
 <text x="86.36" y="21.59" size="1.016" layer="25" ratio="1">+</text>
+<text x="42.164" y="18.542" size="1.016" layer="25" ratio="1">+</text>
+<wire x1="-0.762" y1="9.398" x2="17.018" y2="9.398" width="0.3048" layer="25"/>
 </plain>
 <attributes>
@@
 <element name="JP1" library="SparkFun-Connectors" package="MOLEX-1X2_LOCK" value="M02POLAR_LOCK" x="39.37" y="19.05" smashed="yes" rot="R90"/>
 <element name="JP2" library="SparkFun-Connectors" package="MOLEX-1X2_LOCK" value="M02POLAR_LOCK" x="90.17" y="21.59" smashed="yes" rot="R270"/>
-<element name="Q1" library="transistor-power" package="TO220BV" value="" x="70.104" y="38.1" smashed="yes">
-<attribute name="NAME" x="65.659" y="32.6898" size="0.8128" layer="25" ratio="10"/>
-<attribute name="VALUE" x="65.024" y="30.48" size="1.27" layer="27" ratio="10"/>
+<element name="Q1" library="transistor-power" package="TO220BV" value="" x="71.374" y="38.1" smashed="yes">
+<attribute name="NAME" x="66.929" y="32.6898" size="0.8128" layer="25" ratio="10"/>
+<attribute name="VALUE" x="66.294" y="30.48" size="1.27" layer="27" ratio="10"/>
 </element>
 <element name="R1" library="SparkFun-Resistors" package="1206" value="240" x="53.975" y="27.94" smashed="yes">
@@
 </element>
 <element name="U$2" library="MCP600X" package="SOIC-14" value="MCP6004SOIC" x="68.58" y="24.13" smashed="yes"/>
-<element name="U1" library="v-reg" package="317TS" value=" LD1086BV " x="56.134" y="38.1" smashed="yes"/>
+<element name="U1" library="v-reg" package="317TS" value=" LD1086BV " x="54.864" y="38.1" smashed="yes"/>
 <element name="VREF" library="MCP1525" package="SOT23-3" value="MCP1525/1541SOT" x="54.61" y="15.875" smashed="yes">
 <attribute name="NAME" x="52.832" y="14.4145" size="0.8128" layer="25" rot="R90"/>
@@
 <attribute name="NAME" x="62.357" y="13.97" size="0.8128" layer="25" rot="R90"/>
 </element>
-<element name="C2" library="SparkFun-Capacitors" package="1206" value="10uF" x="44.45" y="20.32" smashed="yes" rot="R90">
-<attribute name="NAME" x="43.307" y="19.05" size="0.8128" layer="25" rot="R90"/>
+<element name="C2" library="SparkFun-Capacitors" package="1206" value="10uF" x="45.974" y="20.32" smashed="yes" rot="R90">
+<attribute name="NAME" x="44.831" y="18.034" size="0.8128" layer="25" rot="R90"/>
 </element>
 <element name="C3" library="SparkFun-Capacitors" package="1206" value="10uF" x="59.055" y="31.496" smashed="yes">
@@
 <contactref element="Q1" pad="S"/>
 <contactref element="C3" pad="1"/>
-<wire x1="56.134" y1="35.56" x2="56.134" y2="33.017" width="1.016" layer="1"/>
-<wire x1="56.134" y1="33.017" x2="57.655" y2="31.496" width="1.016" layer="1"/>
+<wire x1="54.864" y1="34.287" x2="57.655" y2="31.496" width="1.016" layer="1"/>
 <wire x1="57.655" y1="31.496" x2="57.655" y2="30.22" width="1.016" layer="1"/>
 <wire x1="57.655" y1="30.22" x2="55.375" y2="27.94" width="1.016" layer="1"/>
-<wire x1="72.644" y1="35.56" x2="72.644" y2="37.592" width="1.016" layer="1"/>
-<wire x1="72.644" y1="37.592" x2="72.136" y2="38.1" width="1.016" layer="1"/>
-<wire x1="72.136" y1="38.1" x2="56.896" y2="38.1" width="1.016" layer="1"/>
-<wire x1="56.896" y1="38.1" x2="56.134" y2="37.338" width="1.016" layer="1"/>
-<wire x1="56.134" y1="37.338" x2="56.134" y2="35.56" width="1.016" layer="1"/>
+<wire x1="54.864" y1="34.287" x2="54.864" y2="35.56" width="1.016" layer="1"/>
+<wire x1="73.914" y1="35.56" x2="73.914" y2="37.846" width="1.016" layer="1"/>
+<wire x1="73.914" y1="37.846" x2="73.406" y2="38.354" width="1.016" layer="1"/>
+<wire x1="73.406" y1="38.354" x2="55.626" y2="38.354" width="1.016" layer="1"/>
+<wire x1="55.626" y1="38.354" x2="54.864" y2="37.592" width="1.016" layer="1"/>
+<wire x1="54.864" y1="37.592" x2="54.864" y2="35.56" width="1.016" layer="1"/>
 </signal>
 <signal name="VBATT_NEG">
@@
 <contactref element="R8" pad="2"/>
 <contactref element="C2" pad="1"/>
-<wire x1="44.45" y1="18.92" x2="39.373" y2="18.92" width="1.016" layer="1"/>
+<wire x1="45.974" y1="18.92" x2="39.373" y2="18.92" width="1.016" layer="1"/>
 <wire x1="39.373" y1="18.92" x2="39.37" y2="18.923" width="1.016" layer="1"/>
 <wire x1="63.5" y1="17.78" x2="67.31" y2="17.78" width="0.254" layer="1"/>
@@
 <wire x1="67.31" y1="17.78" x2="67.31" y2="17.61" width="0.254" layer="1"/>
 <wire x1="67.945" y1="17.78" x2="67.945" y2="20.8153" width="0.254" layer="1"/>
-<wire x1="58.674" y1="35.56" x2="58.674" y2="24.892" width="1.4224" layer="16"/>
-<wire x1="58.674" y1="24.892" x2="55.88" y2="24.892" width="1.4224" layer="16"/>
+<wire x1="57.404" y1="35.56" x2="57.404" y2="25.146" width="1.4224" layer="16"/>
+<wire x1="57.404" y1="25.146" x2="55.88" y2="24.892" width="1.4224" layer="16"/>
 <wire x1="55.88" y1="24.892" x2="48.006" y2="17.018" width="1.4224" layer="16"/>
 <wire x1="48.006" y1="17.018" x2="41.275" y2="17.018" width="1.4224" layer="16"/>
@@
 <wire x1="54.565" y1="13.97" x2="53.66" y2="14.875" width="0.254" layer="1"/>
 <wire x1="53.66" y1="14.875" x2="48.495" y2="14.875" width="0.254" layer="1"/>
-<wire x1="48.495" y1="14.875" x2="44.45" y2="18.92" width="0.254" layer="1"/>
+<wire x1="48.495" y1="14.875" x2="45.974" y2="18.92" width="0.254" layer="1"/>
 </signal>
 <signal name="N$2">
@@
 <wire x1="52.07" y1="24.26" x2="52.575" y2="24.765" width="0.3048" layer="1"/>
 <wire x1="52.575" y1="24.765" x2="52.575" y2="27.94" width="0.3048" layer="1"/>
-<wire x1="53.594" y1="35.56" x2="53.594" y2="32.001" width="0.3048" layer="1"/>
 <wire x1="53.594" y1="32.001" x2="53.216" y2="31.623" width="0.3048" layer="1"/>
 <wire x1="53.216" y1="31.623" x2="53.216" y2="28.581" width="0.3048" layer="1"/>
 <wire x1="53.216" y1="28.581" x2="52.575" y2="27.94" width="0.3048" layer="1"/>
+<wire x1="53.594" y1="32.001" x2="53.594" y2="32.258" width="0.3048" layer="1"/>
+<wire x1="53.594" y1="32.258" x2="52.324" y2="33.528" width="0.3048" layer="1"/>
+<wire x1="52.324" y1="33.528" x2="52.324" y2="35.56" width="0.3048" layer="1"/>
 </signal>
 <signal name="N$1">
@@
 <wire x1="81.915" y1="29.845" x2="77.089" y2="29.845" width="1.016" layer="1"/>
 <wire x1="77.089" y1="29.845" x2="74.676" y2="32.258" width="1.016" layer="1"/>
-<wire x1="74.676" y1="32.258" x2="70.866" y2="32.258" width="1.016" layer="1"/>
-<wire x1="70.866" y1="32.258" x2="70.104" y2="33.02" width="1.016" layer="1"/>
-<wire x1="70.104" y1="33.02" x2="70.104" y2="35.56" width="1.016" layer="1"/>
+<wire x1="74.676" y1="32.258" x2="72.39" y2="32.258" width="1.016" layer="1"/>
+<wire x1="72.39" y1="32.258" x2="71.374" y2="33.274" width="1.016" layer="1"/>
+<wire x1="71.374" y1="33.274" x2="71.374" y2="35.56" width="1.016" layer="1"/>
 </signal>
 <signal name="ENABLE">
@@
 <wire x1="70.485" y1="16.51" x2="71.12" y2="15.875" width="0.254" layer="1"/>
 <wire x1="70.485" y1="32.131" x2="70.485" y2="16.51" width="0.254" layer="16"/>
-<wire x1="67.564" y1="35.56" x2="70.485" y2="32.131" width="0.254" layer="16"/>
+<wire x1="68.834" y1="35.56" x2="70.485" y2="32.131" width="0.254" layer="16"/>
 <wire x1="71.12" y1="15.875" x2="71.44" y2="15.51" width="0.254" layer="1"/>
 <via x="70.485" y="16.51" extent="1-16" drill="0.254"/>
@@
 <wire x1="77.775" y1="27.381" x2="74.676" y2="30.48" width="0.254" layer="1"/>
 <wire x1="74.676" y1="30.48" x2="70.358" y2="30.48" width="0.254" layer="1"/>
-<wire x1="70.358" y1="30.48" x2="67.564" y2="33.274" width="0.254" layer="1"/>
-<wire x1="67.564" y1="33.274" x2="67.564" y2="35.56" width="0.254" layer="1"/>
+<wire x1="70.358" y1="30.48" x2="68.834" y2="32.004" width="0.254" layer="1"/>
+<wire x1="68.834" y1="32.004" x2="68.834" y2="35.56" width="0.254" layer="1"/>
 </signal>
 <signal name="VREF">
