File: LM317_3S_LithiumCharger_2018_05_13.sch (EAGLE design)
At the start: 27 parts, among them Q2 MOSFET-NCHANNELBSS123LT1G, Q3 MOSFET-PCHANNEL, U1 LD1086BV

Commit message: Add files via upload
Other:
- note added: "12.6V Lithium Charger By Chris Savage 5/13/2018"
Changed lines of the file:
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@@
 7C/W heatsink
 67C </text>
+<text x="60.96" y="60.96" size="1.9304" layer="91">12.6V Lithium Charger
+By Chris Savage
+5/13/2018</text>
 </plain>
 <instances>
